Commit message: Skid Steer Bot equipped with camera and laser

File: mybot_ws(Project)/src/mybot_description/urdf/macros.xacro (robot description, xacro)
@@ -1,22 +1,19 @@
 <?xml version="1.0"?>
 <robot>
-  <!--macro name="cylinder_inertia" params="m r h">
+  <!--xacro:macro name="cylinder_inertia" params="m r h">
     <inertia  ixx="${m*(3*r*r+h*h)/12}" ixy = "0" ixz = "0"
       iyy="${m*(3*r*r+h*h)/12}" iyz = "0"
-      izz="${m*r*r/2}"
-    />
-  </macro>
-  <macro name="box_inertia" params="m x y z">
+      izz="${m*r*r/2}"/>
+  </xacro:macro>
+  <xacro:macro name="box_inertia" params="m x y z">
     <inertia  ixx="${m*(y*y+z*z)/12}" ixy = "0" ixz = "0"
       iyy="${m*(x*x+z*z)/12}" iyz = "0"
-      izz="${m*(x*x+z*z)/12}"
-    />
-  </macro>
-  <macro name="sphere_inertia" params="m r">
+      izz="${m*(x*x+z*z)/12}"/>
+  </xacro:macro>
+  <xacro:macro name="sphere_inertia" params="m r">
     <inertia  ixx="${2*m*r*r/5}" ixy = "0" ixz = "0"
       iyy="${2*m*r*r/5}" iyz = "0"
-      izz="${2*m*r*r/5}"
-    />
-  </macro>
+      izz="${2*m*r*r/5}"/>
+  </xacro:macro>
   <macro name="wheel" params="lr tY">
     <link name="${lr}_wheel">

File: mybot_ws(Project)/src/mybot_description/urdf/mybot.xacro (robot description, xacro)
@@ -6,14 +6,38 @@
   <xacro:include filename="$(find mybot_description)/urdf/materials.xacro" />
   <xacro:include filename="$(find mybot_description)/urdf/macros.xacro" />
+   <xacro:macro name="box_inertia" params="m x y z">
+        <inertial>
+		<origin xyz="0.0 0 0.1" rpy=" 0 0 0"/>
+                <mass value="${m}" />
+                <inertia  ixx="${m*(y*y+z*z)/12}" ixy = "0" ixz = "0"
+      			  iyy="${m*(x*x+z*z)/12}" iyz = "0"
+     			  izz="${m*(x*x+z*z)/12}"/>
+        </inertial>
+   </xacro:macro>
+   <xacro:macro name="cylinder_inertia" params="m r h">
+        <inertial>
+		<origin xyz="0 0 0" rpy="0 1.5707 1.5707"/>
+                <mass value="${m}" />
+                <inertia  ixx="${m*(3*r*r+h*h)/12}" ixy = "0" ixz = "0"
+    			  iyy="${m*(3*r*r+h*h)/12}" iyz = "0"
+    			  izz="${m*r*r/2}"/>
+        </inertial>
+   </xacro:macro>
+   <xacro:macro name="sphere_inertia" params="m x y z">
+        <inertial>
+                <mass value="${m}" />
+                <inertia  ixx="${2*m*r*r/5}" ixy = "0" ixz = "0"
+   			  iyy="${2*m*r*r/5}" iyz = "0"
+     			  izz="${2*m*r*r/5}"/>
+        </inertial>
+   </xacro:macro>
+<!--XXXXXXXXXXXXXXXXXXXXXXXXXXXXXXXXXXXXXXXXXXXXXXXXXXXXXXXXXXXXXXXXXXXXXXXXXXXXXXXXXXXXXXXXXXX-->
   <link name="chassis">
         <pose>0 0 0.1 0 0 0</pose>
-        <inertial>
-            <mass value="20.0"/>
-            <inertia ixx="0.1" ixy="0.0" ixz="0.0" iyy="0.1" iyz="0.0" izz="0.1"/>
-        </inertial>
+     	<xacro:box_inertia m="10" x="0.1" y="0.05" z="0.02"/>
         <visual name="chassis_visual">
             <origin xyz="0.0 0.0 0.0" rpy="0.0 0.0 0.0"/>
             <geometry>
-                <box size="0.1 0.05 0.02"/>
+                <box size="0.1 0.049 0.02"/>
             </geometry>
             <material name="blue"/>
@@ -24,92 +48,4 @@
             </geometry>
         </collision>
- 	   <!--collision name='caster_left_front_collision'>
- 	     <origin xyz="0.045 0.02 -0.01" rpy=" 0 0 0"/>
- 	       <geometry>
-  	         <sphere radius="0.005"/>
-    	       </geometry>
-   	       <surface>
-    	    	 <friction>
-      	     	   <ode>
-     	             <mu>0</mu>
-     	      	     <mu2>0</mu2>
-     	      	     <slip1>1.0</slip1>
-     	      	     <slip2>1.0</slip2>
-      	    	   </ode>
-     	   	</friction>
-    	      </surface>
-   	   </collision>
-  	  <visual name='caster_left_front_visual'>
-   	   <origin xyz="0.045 0.02 -0.01" rpy=" 0 0 0"/>
-    	  <geometry>
-    	    <sphere radius="0.005"/>
-    	  </geometry>
-   	 </visual>
-	 <collision name='caster_left_back_collision'>
- 	     <origin xyz="-0.045 0.02 -0.01" rpy=" 0 0 0"/>
- 	       <geometry>
-  	         <sphere radius="0.005"/>
-    	       </geometry>
-   	       <surface>
-    	    	 <friction>
-      	     	   <ode>
-     	             <mu>0</mu>
-     	      	     <mu2>0</mu2>
-     	      	     <slip1>1.0</slip1>
-     	      	     <slip2>1.0</slip2>
-      	    	   </ode>
-     	   	</friction>
-    	      </surface>
-   	   </collision>
-  	  <visual name='caster_left_back_visual'>
-   	   <origin xyz="-0.045 0.02 -0.01" rpy=" 0 0 0"/>
-    	  <geometry>
-    	    <sphere radius="0.005"/>
-    	  </geometry>
-   	 </visual>
-	 <collision name='caster_right_front_collision'>
- 	     <origin xyz="0.045 -0.02 -0.01" rpy=" 0 0 0"/>
- 	       <geometry>
-  	         <sphere radius="0.005"/>
-    	       </geometry>
-   	       <surface>
-    	    	 <friction>
-      	     	   <ode>
-     	             <mu>0</mu>
-     	      	     <mu2>0</mu2>
-     	      	     <slip1>1.0</slip1>
-     	      	     <slip2>1.0</slip2>
-      	    	   </ode>
-     	   	</friction>
-    	      </surface>
-   	   </collision>
-  	  <visual name='caster_right_front_visual'>
-   	   <origin xyz="0.045 -0.02 -0.01" rpy=" 0 0 0"/>
-    	  <geometry>
-    	    <sphere radius="0.005"/>
-    	  </geometry>
-   	 </visual>
-	  <collision name='caster_right_back_collision'>
- 	     <origin xyz="-0.045 -0.02 -0.01" rpy=" 0 0 0"/>
- 	       <geometry>
-  	         <sphere radius="0.005"/>
-    	       </geometry>
-   	       <surface>
-    	    	 <friction>
-      	     	   <ode>
-     	             <mu>0</mu>
-     	      	     <mu2>0</mu2>
-     	      	     <slip1>1.0</slip1>
-     	      	     <slip2>1.0</slip2>
-      	    	   </ode>
-     	   	</friction>
-    	      </surface>
-   	   </collision>
-  	  <visual name='caster_right_back_visual'>
-   	   <origin xyz="-0.045 -0.02 -0.01" rpy=" 0 0 0"/>
-    	  <geometry>
-    	    <sphere radius="0.005"/>
-    	  </geometry>
-   	 </visual-->
     </link>
     <link name="left_front_wheel">
@@ -126,12 +62,5 @@
             </geometry>
         </visual>
-        <inertial>
-            <origin xyz="0 0 0" rpy="0 1.5707 1.5707"/>
-            <mass value="3"/>
-            <inertia
-                ixx="1.0" ixy="0.0" ixz="0.0"
-                iyy="1.0" iyz="0.0"
-                izz="1.0"/>
-        </inertial>
+        <xacro:cylinder_inertia m="2" r="0.015" h="0.01"/>
     </link>
     <link name="left_back_wheel">
@@ -148,12 +77,5 @@
             </geometry>
         </visual>
-        <inertial>
-            <origin xyz="0 0 0" rpy="0 1.5707 1.5707"/>
-            <mass value="3"/>
-            <inertia
-                ixx="1.0" ixy="0.0" ixz="0.0"
-                iyy="1.0" iyz="0.0"
-                izz="1.0"/>
-        </inertial>
+        <xacro:cylinder_inertia m="2" r="0.015" h="0.01"/>
     </link>
     <link name="right_front_wheel">
@@ -170,12 +92,5 @@
             </geometry>
         </visual>
-        <inertial>
-            <origin xyz="0 0 0" rpy="0 1.5707 1.5707"/>
-            <mass value="3"/>
-            <inertia
-                ixx="1.0" ixy="0.0" ixz="0.0"
-                iyy="1.0" iyz="0.0"
-                izz="1.0"/>
-        </inertial>
+        <xacro:cylinder_inertia m="2" r="0.015" h="0.01"/>
     </link>
     <link name="right_back_wheel">
@@ -192,14 +107,7 @@
             </geometry>
         </visual>
-        <inertial>
-            <origin xyz="0 0 0" rpy="0 1.5707 1.5707"/>
-            <mass value="3"/>
-            <inertia
-                ixx="1.0" ixy="0.0" ixz="0.0"
-                iyy="1.0" iyz="0.0"
-                izz="1.0"/>
-        </inertial>
+        <xacro:cylinder_inertia m="2" r="0.015" h="0.01"/>
     </link>
-    <joint type="continuous" name="left_front_wheel_hinge">
+    <joint type="continuous" name="left_front_wheel_joint">
         <origin xyz="0.03 0.03 0.0" rpy="0 0 0"/>
         <child link="left_front_wheel"/>
@@ -209,5 +117,5 @@
         <joint_properties damping="0.0" friction="0.0"/>
     </joint>
-    <joint type="continuous" name="left_back_wheel_hinge">
+    <joint type="continuous" name="left_back_wheel_joint">
         <origin xyz="-0.03 0.03 0.0" rpy="0 0 0"/>
         <child link="left_back_wheel"/>
@@ -217,5 +125,5 @@
         <joint_properties damping="0.0" friction="0.0"/>
     </joint>
-    <joint type="continuous" name="right_front_wheel_hinge">
+    <joint type="continuous" name="right_front_wheel_joint">
         <origin xyz="0.03 -0.03 0.0" rpy="0 0 0"/>
         <child link="right_front_wheel"/>
@@ -225,5 +133,5 @@
         <joint_properties damping="0.0" friction="0.0"/>
     </joint>
-    <joint type="continuous" name="right_back_wheel_hinge">
+    <joint type="continuous" name="right_back_wheel_joint">
         <origin xyz="-0.03 -0.03 0.0" rpy="0 0 0"/>
         <child link="right_back_wheel"/>
