Commit message: Update on mybot_ws

File: mybot_ws(Project)/src/mybot_description/urdf/mybot.xacro (robot description, xacro)
@@ -8,5 +8,5 @@
    <xacro:macro name="box_inertia" params="m x y z">
         <inertial>
-		<origin xyz="0.0 0 0.1" rpy=" 0 0 0"/>
+		<origin xyz="0.0 0.0 0.1" rpy=" 0 0 0"/>
                 <mass value="${m}" />
                 <inertia  ixx="${m*(y*y+z*z)/12}" ixy = "0" ixz = "0"
@@ -41,5 +41,5 @@
                 <box size="0.1 0.049 0.02"/>
             </geometry>
-            <material name="blue"/>
+            <material name="white"/>
         </visual>
         <collision name='collision'>

Commit message: Control remaining

File: mybot_ws(Project)/src/mybot_description/urdf/mybot.xacro (robot description, xacro)
@@ -45,5 +45,5 @@
         <collision name='collision'>
             <geometry>
-                <box size="0.1 0.05 0.02"/>
+                <box size="0.1 0.049 0.02"/>
             </geometry>
         </collision>
@@ -62,5 +62,5 @@
             </geometry>
         </visual>
-        <xacro:cylinder_inertia m="2" r="0.015" h="0.01"/>
+        <xacro:cylinder_inertia m="0.5" r="0.015" h="0.01"/>
     </link>
     <link name="left_back_wheel">
@@ -77,5 +77,5 @@
             </geometry>
         </visual>
-        <xacro:cylinder_inertia m="2" r="0.015" h="0.01"/>
+        <xacro:cylinder_inertia m="0.5" r="0.015" h="0.01"/>
     </link>
     <link name="right_front_wheel">
@@ -92,5 +92,5 @@
             </geometry>
         </visual>
-        <xacro:cylinder_inertia m="2" r="0.015" h="0.01"/>
+        <xacro:cylinder_inertia m="0.5" r="0.015" h="0.01"/>
     </link>
     <link name="right_back_wheel">
@@ -107,5 +107,5 @@
             </geometry>
         </visual>
-        <xacro:cylinder_inertia m="2" r="0.015" h="0.01"/>
+        <xacro:cylinder_inertia m="0.5" r="0.015" h="0.01"/>
     </link>
     <joint type="continuous" name="left_front_wheel_joint">

Commit message: Closed room added +Modifications on the bot

File: mybot_ws(Project)/src/mybot_description/urdf/mybot.xacro (robot description, xacro)
@@ -49,4 +49,24 @@
         </collision>
     </link>
+      <link name="stand">
+     	<xacro:box_inertia m="1" x="0.03" y="0.03" z="0.09"/>
+        <visual name="chassis_visual">
+            <origin xyz="0.0 0.0 0.0" rpy="0.0 0.0 0.0"/>
+            <geometry>
+                <box size="0.03 0.03 0.09"/>
+            </geometry>
+            <material name="white"/>
+        </visual>
+        <collision name='collision'>
+            <geometry>
+                <box size="0.03 0.03 0.09"/>
+            </geometry>
+        </collision>
+    </link>
+  <joint name="stand_joint" type="fixed">
+    <parent link="chassis"/>
+    <child link="stand"/>
+    <origin xyz="0 0 0.05"/>
+  </joint>
     <link name="left_front_wheel">
         <collision name="collision">
@@ -115,5 +135,5 @@
         <axis xyz="0 1 0" rpy="0 0 0"/>
         <limit effort="100" velocity="100"/>
-        <joint_properties damping="0.0" friction="0.0"/>
+        <joint_properties damping="1.0" friction="0.0"/>
     </joint>
     <joint type="continuous" name="left_back_wheel_joint">
@@ -123,5 +143,5 @@
         <axis xyz="0 1 0" rpy="0 0 0"/>
         <limit effort="100" velocity="100"/>
-        <joint_properties damping="0.0" friction="0.0"/>
+        <joint_properties damping="1.0" friction="0.0"/>
     </joint>
     <joint type="continuous" name="right_front_wheel_joint">
@@ -131,5 +151,5 @@
         <axis xyz="0 1 0" rpy="0 0 0"/>
         <limit effort="100" velocity="100"/>
-        <joint_properties damping="0.0" friction="0.0"/>
+        <joint_properties damping="1.0" friction="0.0"/>
     </joint>
     <joint type="continuous" name="right_back_wheel_joint">
@@ -139,5 +159,5 @@
         <axis xyz="0 1 0" rpy="0 0 0"/>
         <limit effort="100" velocity="100"/>
-        <joint_properties damping="0.0" friction="0.0"/>
+        <joint_properties damping="1.0" friction="0.0"/>
     </joint>
   <link name="camera">
@@ -170,5 +190,5 @@
   <joint name="hokuyo_joint" type="fixed">
     <axis xyz="0 1 0" />
-    <origin xyz="0 0 0.02" rpy="0 0 0"/>
+    <origin xyz="0 0 0.1" rpy="0 0 0"/>
     <parent link="chassis"/>
     <child link="hokuyo"/>

Commit message: Room1 + Maze added

File: mybot_ws(Project)/src/mybot_description/urdf/mybot.xacro (robot description, xacro)
@@ -8,5 +8,5 @@
    <xacro:macro name="box_inertia" params="m x y z">
         <inertial>
-		<origin xyz="0.0 0 0.1" rpy=" 0 0 0"/>
+		<origin xyz="0.0 0.0 0.1" rpy=" 0 0 0"/>
                 <mass value="${m}" />
                 <inertia  ixx="${m*(y*y+z*z)/12}" ixy = "0" ixz = "0"
@@ -41,12 +41,32 @@
                 <box size="0.1 0.049 0.02"/>
             </geometry>
-            <material name="blue"/>
+            <material name="white"/>
         </visual>
         <collision name='collision'>
             <geometry>
-                <box size="0.1 0.05 0.02"/>
-            </geometry>
-        </collision>
-    </link>
+                <box size="0.1 0.049 0.02"/>
+            </geometry>
+        </collision>
+    </link>
+      <link name="stand">
+     	<xacro:box_inertia m="5" x="0.03" y="0.03" z="0.09"/>
+        <visual name="chassis_visual">
+            <origin xyz="0.0 0.0 0.0" rpy="0.0 0.0 0.0"/>
+            <geometry>
+                <box size="0.03 0.03 0.09"/>
+            </geometry>
+            <material name="white"/>
+        </visual>
+        <collision name='collision'>
+            <geometry>
+                <box size="0.03 0.03 0.09"/>
+            </geometry>
+        </collision>
+    </link>
+  <joint name="stand_joint" type="fixed">
+    <parent link="chassis"/>
+    <child link="stand"/>
+    <origin xyz="0 0 0.05"/>
+  </joint>
     <link name="left_front_wheel">
         <collision name="collision">
@@ -62,5 +82,5 @@
             </geometry>
         </visual>
-        <xacro:cylinder_inertia m="2" r="0.015" h="0.01"/>
+        <xacro:cylinder_inertia m="1" r="0.015" h="0.01"/>
     </link>
     <link name="left_back_wheel">
@@ -77,5 +97,5 @@
             </geometry>
         </visual>
-        <xacro:cylinder_inertia m="2" r="0.015" h="0.01"/>
+        <xacro:cylinder_inertia m="1" r="0.015" h="0.01"/>
     </link>
     <link name="right_front_wheel">
@@ -92,5 +112,5 @@
             </geometry>
         </visual>
-        <xacro:cylinder_inertia m="2" r="0.015" h="0.01"/>
+        <xacro:cylinder_inertia m="1" r="0.015" h="0.01"/>
     </link>
     <link name="right_back_wheel">
@@ -107,5 +127,5 @@
             </geometry>
         </visual>
-        <xacro:cylinder_inertia m="2" r="0.015" h="0.01"/>
+        <xacro:cylinder_inertia m="1" r="0.015" h="0.01"/>
     </link>
     <joint type="continuous" name="left_front_wheel_joint">
@@ -115,5 +135,5 @@
         <axis xyz="0 1 0" rpy="0 0 0"/>
         <limit effort="100" velocity="100"/>
-        <joint_properties damping="0.0" friction="0.0"/>
+        <joint_properties damping="1.0" friction="0.0"/>
     </joint>
     <joint type="continuous" name="left_back_wheel_joint">
@@ -123,5 +143,5 @@
         <axis xyz="0 1 0" rpy="0 0 0"/>
         <limit effort="100" velocity="100"/>
-        <joint_properties damping="0.0" friction="0.0"/>
+        <joint_properties damping="1.0" friction="0.0"/>
     </joint>
     <joint type="continuous" name="right_front_wheel_joint">
@@ -131,5 +151,5 @@
         <axis xyz="0 1 0" rpy="0 0 0"/>
         <limit effort="100" velocity="100"/>
-        <joint_properties damping="0.0" friction="0.0"/>
+        <joint_properties damping="1.0" friction="0.0"/>
     </joint>
     <joint type="continuous" name="right_back_wheel_joint">
@@ -139,5 +159,5 @@
         <axis xyz="0 1 0" rpy="0 0 0"/>
         <limit effort="100" velocity="100"/>
-        <joint_properties damping="0.0" friction="0.0"/>
+        <joint_properties damping="1.0" friction="0.0"/>
     </joint>
   <link name="camera">
@@ -170,5 +190,5 @@
   <joint name="hokuyo_joint" type="fixed">
     <axis xyz="0 1 0" />
-    <origin xyz="0 0 0.02" rpy="0 0 0"/>
+    <origin xyz="0 0 0.1" rpy="0 0 0"/>
     <parent link="chassis"/>
     <child link="hokuyo"/>

Commit message: Room1 + Maze added

File: mybot_ws(Project)/src/mybot_description/urdf/mybot.xacro (robot description, xacro)
@@ -49,4 +49,24 @@
         </collision>
     </link>
+      <link name="stand">
+     	<xacro:box_inertia m="5" x="0.03" y="0.03" z="0.09"/>
+        <visual name="chassis_visual">
+            <origin xyz="0.0 0.0 0.0" rpy="0.0 0.0 0.0"/>
+            <geometry>
+                <box size="0.03 0.03 0.09"/>
+            </geometry>
+            <material name="white"/>
+        </visual>
+        <collision name='collision'>
+            <geometry>
+                <box size="0.03 0.03 0.09"/>
+            </geometry>
+        </collision>
+    </link>
+  <joint name="stand_joint" type="fixed">
+    <parent link="chassis"/>
+    <child link="stand"/>
+    <origin xyz="0 0 0.05"/>
+  </joint>
     <link name="left_front_wheel">
         <collision name="collision">
@@ -62,5 +82,5 @@
             </geometry>
         </visual>
-        <xacro:cylinder_inertia m="0.5" r="0.015" h="0.01"/>
+        <xacro:cylinder_inertia m="1" r="0.015" h="0.01"/>
     </link>
     <link name="left_back_wheel">
@@ -77,5 +97,5 @@
             </geometry>
         </visual>
-        <xacro:cylinder_inertia m="0.5" r="0.015" h="0.01"/>
+        <xacro:cylinder_inertia m="1" r="0.015" h="0.01"/>
     </link>
     <link name="right_front_wheel">
@@ -92,5 +112,5 @@
             </geometry>
         </visual>
-        <xacro:cylinder_inertia m="0.5" r="0.015" h="0.01"/>
+        <xacro:cylinder_inertia m="1" r="0.015" h="0.01"/>
     </link>
     <link name="right_back_wheel">
@@ -107,5 +127,5 @@
             </geometry>
         </visual>
-        <xacro:cylinder_inertia m="0.5" r="0.015" h="0.01"/>
+        <xacro:cylinder_inertia m="1" r="0.015" h="0.01"/>
     </link>
     <joint type="continuous" name="left_front_wheel_joint">
@@ -115,5 +135,5 @@
         <axis xyz="0 1 0" rpy="0 0 0"/>
         <limit effort="100" velocity="100"/>
-        <joint_properties damping="0.0" friction="0.0"/>
+        <joint_properties damping="1.0" friction="0.0"/>
     </joint>
     <joint type="continuous" name="left_back_wheel_joint">
@@ -123,5 +143,5 @@
         <axis xyz="0 1 0" rpy="0 0 0"/>
         <limit effort="100" velocity="100"/>
-        <joint_properties damping="0.0" friction="0.0"/>
+        <joint_properties damping="1.0" friction="0.0"/>
     </joint>
     <joint type="continuous" name="right_front_wheel_joint">
@@ -131,5 +151,5 @@
         <axis xyz="0 1 0" rpy="0 0 0"/>
         <limit effort="100" velocity="100"/>
-        <joint_properties damping="0.0" friction="0.0"/>
+        <joint_properties damping="1.0" friction="0.0"/>
     </joint>
     <joint type="continuous" name="right_back_wheel_joint">
@@ -139,5 +159,5 @@
         <axis xyz="0 1 0" rpy="0 0 0"/>
         <limit effort="100" velocity="100"/>
-        <joint_properties damping="0.0" friction="0.0"/>
+        <joint_properties damping="1.0" friction="0.0"/>
     </joint>
   <link name="camera">
@@ -170,5 +190,5 @@
   <joint name="hokuyo_joint" type="fixed">
     <axis xyz="0 1 0" />
-    <origin xyz="0 0 0.02" rpy="0 0 0"/>
+    <origin xyz="0 0 0.1" rpy="0 0 0"/>
     <parent link="chassis"/>
     <child link="hokuyo"/>

Commit message: Smoothened control

File: mybot_ws(Project)/src/mybot_description/urdf/mybot.xacro (robot description, xacro)
@@ -34,5 +34,5 @@
 <!--XXXXXXXXXXXXXXXXXXXXXXXXXXXXXXXXXXXXXXXXXXXXXXXXXXXXXXXXXXXXXXXXXXXXXXXXXXXXXXXXXXXXXXXXXXX-->
   <link name="chassis">
-        <pose>0 0 0.1 0 0 0</pose>
+        <pose>0 0 0.2 0 0 0</pose>
      	<xacro:box_inertia m="10" x="0.1" y="0.05" z="0.02"/>
         <visual name="chassis_visual">
@@ -49,24 +49,4 @@
         </collision>
     </link>
-      <link name="stand">
-     	<xacro:box_inertia m="5" x="0.03" y="0.03" z="0.09"/>
-        <visual name="chassis_visual">
-            <origin xyz="0.0 0.0 0.0" rpy="0.0 0.0 0.0"/>
-            <geometry>
-                <box size="0.03 0.03 0.09"/>
-            </geometry>
-            <material name="white"/>
-        </visual>
-        <collision name='collision'>
-            <geometry>
-                <box size="0.03 0.03 0.09"/>
-            </geometry>
-        </collision>
-    </link>
-  <joint name="stand_joint" type="fixed">
-    <parent link="chassis"/>
-    <child link="stand"/>
-    <origin xyz="0 0 0.05"/>
-  </joint>
     <link name="left_front_wheel">
         <collision name="collision">
@@ -190,5 +170,5 @@
   <joint name="hokuyo_joint" type="fixed">
     <axis xyz="0 1 0" />
-    <origin xyz="0 0 0.1" rpy="0 0 0"/>
+    <origin xyz="0 0 0.02" rpy="0 0 0"/>
     <parent link="chassis"/>
     <child link="hokuyo"/>
@@ -199,5 +179,5 @@
       <origin xyz="0 0 0" rpy="0 0 0"/>
       <geometry>
-    <box size="0.01 0.01 0.01"/>
+    <box size="0.01 0.01 0.02"/>
       </geometry>
     </collision>
@@ -211,5 +191,5 @@
       <mass value="1e-5" />
       <origin xyz="0 0 0" rpy="0 0 0"/>
-      <inertia ixx="1e-6" ixy="0" ixz="0" iyy="1e-6" iyz="0" izz="1e-6" />
+      <inertia ixx="0.1" ixy="0" ixz="0" iyy="0.1" iyz="0" izz="0.01" />
     </inertial>
   </link>

Commit message: updated

File: mybot_ws(Project)/src/mybot_description/urdf/mybot.xacro (robot description, xacro)
@@ -34,5 +34,5 @@
 <!--XXXXXXXXXXXXXXXXXXXXXXXXXXXXXXXXXXXXXXXXXXXXXXXXXXXXXXXXXXXXXXXXXXXXXXXXXXXXXXXXXXXXXXXXXXX-->
   <link name="chassis">
-        <pose>0 0 0.1 0 0 0</pose>
+        <pose>0 0 0.2 0 0 0</pose>
      	<xacro:box_inertia m="10" x="0.1" y="0.05" z="0.02"/>
         <visual name="chassis_visual">
@@ -49,24 +49,4 @@
         </collision>
     </link>
-      <link name="stand">
-     	<xacro:box_inertia m="5" x="0.03" y="0.03" z="0.09"/>
-        <visual name="chassis_visual">
-            <origin xyz="0.0 0.0 0.0" rpy="0.0 0.0 0.0"/>
-            <geometry>
-                <box size="0.03 0.03 0.09"/>
-            </geometry>
-            <material name="white"/>
-        </visual>
-        <collision name='collision'>
-            <geometry>
-                <box size="0.03 0.03 0.09"/>
-            </geometry>
-        </collision>
-    </link>
-  <joint name="stand_joint" type="fixed">
-    <parent link="chassis"/>
-    <child link="stand"/>
-    <origin xyz="0 0 0.05"/>
-  </joint>
     <link name="left_front_wheel">
         <collision name="collision">
@@ -161,4 +141,41 @@
         <joint_properties damping="1.0" friction="0.0"/>
     </joint>
+    <!--experiment-->
+    <!--transmission name="front_right_wheel_trans" type="SimpleTransmission">
+    <type>transmission_interface/SimpleTransmission</type>
+    <actuator name="front_right_wheel_motor">
+      <mechanicalReduction>1</mechanicalReduction>
+    </actuator>
+    <joint name="right_front_wheel_joint">
+      <hardwareInterface>hardware_interface/EffortJointInterface</hardwareInterface>
+    </joint>
+  </transmission>
+  <transmission name="back_right_wheel_trans" type="SimpleTransmission">
+    <type>transmission_interface/SimpleTransmission</type>
+    <actuator name="back_right_wheel_motor">
+      <mechanicalReduction>1</mechanicalReduction>
+    </actuator>
+    <joint name="right_back_wheel_joint">
+      <hardwareInterface>hardware_interface/EffortJointInterface</hardwareInterface>
+    </joint>
+  </transmission>
+  <transmission name="front_left_wheel_trans" type="SimpleTransmission">
+    <type>transmission_interface/SimpleTransmission</type>
+    <actuator name="front_left_wheel_motor">
+      <mechanicalReduction>1</mechanicalReduction>
+    </actuator>
+    <joint name="left_front_wheel_joint">
+      <hardwareInterface>hardware_interface/EffortJointInterface</hardwareInterface>
+    </joint>
+  </transmission>
+  <transmission name="back_left_wheel_trans" type="SimpleTransmission">
+    <type>transmission_interface/SimpleTransmission</type>
+    <actuator name="back_left_wheel_motor">
+      <mechanicalReduction>1</mechanicalReduction>
+    </actuator>
+    <joint name="left_back_wheel_joint">
+      <hardwareInterface>hardware_interface/EffortJointInterface</hardwareInterface>
+    </joint>
+  </transmission-->
   <link name="camera">
     <collision>
@@ -190,5 +207,5 @@
   <joint name="hokuyo_joint" type="fixed">
     <axis xyz="0 1 0" />
-    <origin xyz="0 0 0.1" rpy="0 0 0"/>
+    <origin xyz="0 0 0.02" rpy="0 0 0"/>
     <parent link="chassis"/>
     <child link="hokuyo"/>
@@ -199,5 +216,5 @@
       <origin xyz="0 0 0" rpy="0 0 0"/>
       <geometry>
-    <box size="0.01 0.01 0.01"/>
+    <box size="0.01 0.01 0.02"/>
       </geometry>
     </collision>
@@ -211,5 +228,5 @@
       <mass value="1e-5" />
       <origin xyz="0 0 0" rpy="0 0 0"/>
-      <inertia ixx="1e-6" ixy="0" ixz="0" iyy="1e-6" iyz="0" izz="1e-6" />
+      <inertia ixx="0.1" ixy="0" ixz="0" iyy="0.1" iyz="0" izz="0.01" />
     </inertial>
   </link>

Commit message: updates

File: mybot_ws(Project)/src/mybot_description/urdf/mybot.xacro (robot description, xacro)
@@ -141,4 +141,41 @@
         <joint_properties damping="1.0" friction="0.0"/>
     </joint>
+    <!--experiment-->
+    <!--transmission name="front_right_wheel_trans" type="SimpleTransmission">
+    <type>transmission_interface/SimpleTransmission</type>
+    <actuator name="front_right_wheel_motor">
+      <mechanicalReduction>1</mechanicalReduction>
+    </actuator>
+    <joint name="right_front_wheel_joint">
+      <hardwareInterface>hardware_interface/EffortJointInterface</hardwareInterface>
+    </joint>
+  </transmission>
+  <transmission name="back_right_wheel_trans" type="SimpleTransmission">
+    <type>transmission_interface/SimpleTransmission</type>
+    <actuator name="back_right_wheel_motor">
+      <mechanicalReduction>1</mechanicalReduction>
+    </actuator>
+    <joint name="right_back_wheel_joint">
+      <hardwareInterface>hardware_interface/EffortJointInterface</hardwareInterface>
+    </joint>
+  </transmission>
+  <transmission name="front_left_wheel_trans" type="SimpleTransmission">
+    <type>transmission_interface/SimpleTransmission</type>
+    <actuator name="front_left_wheel_motor">
+      <mechanicalReduction>1</mechanicalReduction>
+    </actuator>
+    <joint name="left_front_wheel_joint">
+      <hardwareInterface>hardware_interface/EffortJointInterface</hardwareInterface>
+    </joint>
+  </transmission>
+  <transmission name="back_left_wheel_trans" type="SimpleTransmission">
+    <type>transmission_interface/SimpleTransmission</type>
+    <actuator name="back_left_wheel_motor">
+      <mechanicalReduction>1</mechanicalReduction>
+    </actuator>
+    <joint name="left_back_wheel_joint">
+      <hardwareInterface>hardware_interface/EffortJointInterface</hardwareInterface>
+    </joint>
+  </transmission-->
   <link name="camera">
     <collision>
