Commit message: Camera Orientation

File: mybot_ws(Project)/src/mybot_description/urdf/mybot.xacro (robot description, xacro)
@@ -1,6 +1,6 @@
 <?xml version='1.0'?>
 <robot name="myrobot" xmlns:xacro="http://www.ros.org/wiki/xacro">
-  <xacro:property name="cameraSize" value="0.015"/>
-  <xacro:property name="cameraMass" value="0.1"/>
+  <xacro:property name="cameraSize" value="0.01"/>
+  <xacro:property name="cameraMass" value="0.01"/>
   <xacro:include filename="$(find mybot_description)/urdf/mybot.gazebo" />
   <xacro:include filename="$(find mybot_description)/urdf/materials.xacro" />
@@ -35,5 +35,5 @@
   <link name="chassis">
         <pose>0 0 0.2 0 0 0</pose>
-     	<xacro:box_inertia m="10" x="0.1" y="0.05" z="0.02"/>
+     	<xacro:box_inertia m="2" x="0.1" y="0.05" z="0.02"/>
         <visual name="chassis_visual">
             <origin xyz="0.0 0.0 0.0" rpy="0.0 0.0 0.0"/>
@@ -62,5 +62,5 @@
             </geometry>
         </visual>
-        <xacro:cylinder_inertia m="1" r="0.015" h="0.01"/>
+        <xacro:cylinder_inertia m="0.3" r="0.015" h="0.01"/>
     </link>
     <link name="left_back_wheel">
@@ -77,5 +77,5 @@
             </geometry>
         </visual>
-        <xacro:cylinder_inertia m="1" r="0.015" h="0.01"/>
+        <xacro:cylinder_inertia m="0.3" r="0.015" h="0.01"/>
     </link>
     <link name="right_front_wheel">
@@ -92,5 +92,5 @@
             </geometry>
         </visual>
-        <xacro:cylinder_inertia m="1" r="0.015" h="0.01"/>
+        <xacro:cylinder_inertia m="0.3" r="0.015" h="0.01"/>
     </link>
     <link name="right_back_wheel">
@@ -107,5 +107,5 @@
             </geometry>
         </visual>
-        <xacro:cylinder_inertia m="1" r="0.015" h="0.01"/>
+        <xacro:cylinder_inertia m="0.3" r="0.015" h="0.01"/>
     </link>
     <joint type="continuous" name="left_front_wheel_joint">
@@ -141,41 +141,4 @@
         <joint_properties damping="1.0" friction="0.0"/>
     </joint>
-    <!--experiment-->
-    <!--transmission name="front_right_wheel_trans" type="SimpleTransmission">
-    <type>transmission_interface/SimpleTransmission</type>
-    <actuator name="front_right_wheel_motor">
-      <mechanicalReduction>1</mechanicalReduction>
-    </actuator>
-    <joint name="right_front_wheel_joint">
-      <hardwareInterface>hardware_interface/EffortJointInterface</hardwareInterface>
-    </joint>
-  </transmission>
-  <transmission name="back_right_wheel_trans" type="SimpleTransmission">
-    <type>transmission_interface/SimpleTransmission</type>
-    <actuator name="back_right_wheel_motor">
-      <mechanicalReduction>1</mechanicalReduction>
-    </actuator>
-    <joint name="right_back_wheel_joint">
-      <hardwareInterface>hardware_interface/EffortJointInterface</hardwareInterface>
-    </joint>
-  </transmission>
-  <transmission name="front_left_wheel_trans" type="SimpleTransmission">
-    <type>transmission_interface/SimpleTransmission</type>
-    <actuator name="front_left_wheel_motor">
-      <mechanicalReduction>1</mechanicalReduction>
-    </actuator>
-    <joint name="left_front_wheel_joint">
-      <hardwareInterface>hardware_interface/EffortJointInterface</hardwareInterface>
-    </joint>
-  </transmission>
-  <transmission name="back_left_wheel_trans" type="SimpleTransmission">
-    <type>transmission_interface/SimpleTransmission</type>
-    <actuator name="back_left_wheel_motor">
-      <mechanicalReduction>1</mechanicalReduction>
-    </actuator>
-    <joint name="left_back_wheel_joint">
-      <hardwareInterface>hardware_interface/EffortJointInterface</hardwareInterface>
-    </joint>
-  </transmission-->
   <link name="camera">
     <collision>
@@ -196,10 +159,10 @@
       <origin xyz="0 0 0" rpy="0 0 0"/>
       <box_inertia m="${cameraMass}" x="${cameraSize}" y="${cameraSize}" z="${cameraSize}" />
-      <inertia ixx="1e-6" ixy="0" ixz="0" iyy="1e-6" iyz="0" izz="1e-6" />
+      <inertia ixx="0.001" ixy="0" ixz="0" iyy="0.001" iyz="0" izz="0.001" />
     </inertial>
   </link>
   <joint name="camera_joint" type="fixed">
     <axis xyz="0 1 0" />
-    <origin xyz="0.05 0 0" rpy="0 0 0"/>
+    <origin xyz="0 0.025 0" rpy="0 0 1.570796"/>
     <parent link="chassis"/>
     <child link="camera"/>
@@ -226,8 +189,48 @@
     </visual>
     <inertial>
-      <mass value="1e-5" />
+      <mass value="0.01" />
       <origin xyz="0 0 0" rpy="0 0 0"/>
       <inertia ixx="0.1" ixy="0" ixz="0" iyy="0.1" iyz="0" izz="0.01" />
     </inertial>
   </link>
+  <!--transmission name="tran1">
+    <type>transmission_interface/SimpleTransmission</type>
+    <joint name="left_front_wheel_joint">
+      <hardwareInterface>EffortJointInterface</hardwareInterface>
+    </joint>
+    <actuator name="motor1">
+      <hardwareInterface>EffortJointInterface</hardwareInterface>
+      <mechanicalReduction>1</mechanicalReduction>
+    </actuator>
+  </transmission>
+  <transmission name="tran2">
+    <type>transmission_interface/SimpleTransmission</type>
+    <joint name="right_front_wheel_joint">
+      <hardwareInterface>EffortJointInterface</hardwareInterface>
+    </joint>
+    <actuator name="motor2">
+      <hardwareInterface>EffortJointInterface</hardwareInterface>
+      <mechanicalReduction>1</mechanicalReduction>
+    </actuator>
+  </transmission>
+  <transmission name="tran3">
+    <type>transmission_interface/SimpleTransmission</type>
+    <joint name="left_back_wheel_joint">
+      <hardwareInterface>EffortJointInterface</hardwareInterface>
+    </joint>
+    <actuator name="motor3">
+      <hardwareInterface>EffortJointInterface</hardwareInterface>
+      <mechanicalReduction>1</mechanicalReduction>
+    </actuator>
+  </transmission>
+  <transmission name="tran4">
+    <type>transmission_interface/SimpleTransmission</type>
+    <joint name="right_back_wheel_joint">
+      <hardwareInterface>EffortJointInterface</hardwareInterface>
+    </joint>
+    <actuator name="motor4">
+      <hardwareInterface>EffortJointInterface</hardwareInterface>
+      <mechanicalReduction>1</mechanicalReduction>
+    </actuator>
+  </transmission-->
 </robot>

Commit message: The Master-Merge

File: mybot_ws(Project)/src/mybot_description/urdf/mybot.xacro (robot description, xacro)
@@ -159,5 +159,5 @@
       <origin xyz="0 0 0" rpy="0 0 0"/>
       <box_inertia m="${cameraMass}" x="${cameraSize}" y="${cameraSize}" z="${cameraSize}" />
-      <inertia ixx="0.001" ixy="0" ixz="0" iyy="0.001" iyz="0" izz="0.001" />
+      <inertia ixx="0.1" ixy="0" ixz="0" iyy="0.1" iyz="0" izz="0.1" />
     </inertial>
   </link>
@@ -191,5 +191,5 @@
       <mass value="0.01" />
       <origin xyz="0 0 0" rpy="0 0 0"/>
-      <inertia ixx="0.1" ixy="0" ixz="0" iyy="0.1" iyz="0" izz="0.01" />
+      <inertia ixx="0.1" ixy="0" ixz="0" iyy="0.1" iyz="0" izz="0.1" />
     </inertial>
   </link>

Commit message: minor changes

File: mybot_ws(Project)/src/mybot_description/urdf/mybot.xacro (robot description, xacro)
@@ -1,5 +1,5 @@
 <?xml version='1.0'?>
 <robot name="myrobot" xmlns:xacro="http://www.ros.org/wiki/xacro">
-  <xacro:property name="cameraSize" value="0.01"/>
+  <xacro:property name="cameraSize" value="0.006"/>
   <xacro:property name="cameraMass" value="0.01"/>
   <xacro:include filename="$(find mybot_description)/urdf/mybot.gazebo" />
@@ -35,5 +35,5 @@
   <link name="chassis">
         <pose>0 0 0.2 0 0 0</pose>
-     	<xacro:box_inertia m="2" x="0.1" y="0.05" z="0.02"/>
+     	<xacro:box_inertia m="1.5" x="0.1" y="0.05" z="0.02"/>
         <visual name="chassis_visual">
             <origin xyz="0.0 0.0 0.0" rpy="0.0 0.0 0.0"/>
@@ -62,5 +62,5 @@
             </geometry>
         </visual>
-        <xacro:cylinder_inertia m="0.3" r="0.015" h="0.01"/>
+        <xacro:cylinder_inertia m="0.5" r="0.015" h="0.01"/>
     </link>
     <link name="left_back_wheel">
@@ -77,5 +77,5 @@
             </geometry>
         </visual>
-        <xacro:cylinder_inertia m="0.3" r="0.015" h="0.01"/>
+        <xacro:cylinder_inertia m="0.5" r="0.015" h="0.01"/>
     </link>
     <link name="right_front_wheel">
@@ -92,5 +92,5 @@
             </geometry>
         </visual>
-        <xacro:cylinder_inertia m="0.3" r="0.015" h="0.01"/>
+        <xacro:cylinder_inertia m="0.5" r="0.015" h="0.01"/>
     </link>
     <link name="right_back_wheel">
@@ -107,5 +107,5 @@
             </geometry>
         </visual>
-        <xacro:cylinder_inertia m="0.3" r="0.015" h="0.01"/>
+        <xacro:cylinder_inertia m="0.5" r="0.015" h="0.01"/>
     </link>
     <joint type="continuous" name="left_front_wheel_joint">
@@ -164,5 +164,5 @@
   <joint name="camera_joint" type="fixed">
     <axis xyz="0 1 0" />
-    <origin xyz="0 0.025 0" rpy="0 0 1.570796"/>
+    <origin xyz="0 0.0215 0.013" rpy="0 0 1.570796"/>
     <parent link="chassis"/>
     <child link="camera"/>
@@ -189,5 +189,5 @@
     </visual>
     <inertial>
-      <mass value="0.01" />
+      <mass value="0.05" />
       <origin xyz="0 0 0" rpy="0 0 0"/>
       <inertia ixx="0.1" ixy="0" ixz="0" iyy="0.1" iyz="0" izz="0.1" />

Commit message: Wall Follower Final Edit

File: mybot_ws(Project)/src/mybot_description/urdf/mybot.xacro (robot description, xacro)
@@ -39,5 +39,5 @@
             <origin xyz="0.0 0.0 0.0" rpy="0.0 0.0 0.0"/>
             <geometry>
-                <box size="0.1 0.049 0.02"/>
+                <box size="0.08 0.049 0.02"/>
             </geometry>
             <material name="white"/>
@@ -45,5 +45,5 @@
         <collision name='collision'>
             <geometry>
-                <box size="0.1 0.049 0.02"/>
+                <box size="0.08 0.049 0.02"/>
             </geometry>
         </collision>
@@ -110,5 +110,5 @@
     </link>
     <joint type="continuous" name="left_front_wheel_joint">
-        <origin xyz="0.03 0.03 0.0" rpy="0 0 0"/>
+        <origin xyz="0.02 0.03 0.0" rpy="0 0 0"/>
         <child link="left_front_wheel"/>
         <parent link="chassis"/>
@@ -118,5 +118,5 @@
     </joint>
     <joint type="continuous" name="left_back_wheel_joint">
-        <origin xyz="-0.03 0.03 0.0" rpy="0 0 0"/>
+        <origin xyz="-0.02 0.03 0.0" rpy="0 0 0"/>
         <child link="left_back_wheel"/>
         <parent link="chassis"/>
@@ -126,5 +126,5 @@
     </joint>
     <joint type="continuous" name="right_front_wheel_joint">
-        <origin xyz="0.03 -0.03 0.0" rpy="0 0 0"/>
+        <origin xyz="0.02 -0.03 0.0" rpy="0 0 0"/>
         <child link="right_front_wheel"/>
         <parent link="chassis"/>
@@ -134,5 +134,5 @@
     </joint>
     <joint type="continuous" name="right_back_wheel_joint">
-        <origin xyz="-0.03 -0.03 0.0" rpy="0 0 0"/>
+        <origin xyz="-0.02 -0.03 0.0" rpy="0 0 0"/>
         <child link="right_back_wheel"/>
         <parent link="chassis"/>
